File: KiCAD/21FX/21FX.kicad_sch (KiCad schematic)
At the start: 12 parts, among them J1 DB25_Socket_MountingHoles, J2 SST39SF040, J3 Adafruit 232H, J4 Altera JTAG, J5 Select 5v, U1 EPM7064STC44-10, X1 ASDMB-xxxMHz

Commit message: Add files via upload
Parts:
- X1: value ASDMB-xxxMHz -> CTX314CT-ND 40mhz; footprint Oscillator:Oscillator_SMD_Abracon_ASDMB-4Pin_2.5x2.0mm -> Oscillator:Oscillator_SMD_Abracon_ASV-4Pin_7.0x5.1mm
Changed lines of the file:
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@@
 		(on_board yes)
 		(dnp no)
-		(fields_autoplaced yes)
 		(property "Reference" "X1"
 			(at 120.65 26.5998 0)
@@
 			)
 		)
-		(property "Value" "ASDMB-xxxMHz"
-			(at 120.65 29.1398 0)
+		(property "Value" "CTX314CT-ND 40mhz"
+			(at 106.68 41.148 0)
 			(effects
 				(font
@@
 			)
 		)
-		(property "Footprint" "Oscillator:Oscillator_SMD_Abracon_ASDMB-4Pin_2.5x2.0mm"
+		(property "Footprint" "Oscillator:Oscillator_SMD_Abracon_ASV-4Pin_7.0x5.1mm"
 			(at 104.14 33.02 0)
 			(effects
