File: KiCAD/21FX/21FX.kicad_pcb (KiCad board)
At the start: 4 copper layers, 53.5 x 34.9 mm, 12 parts, among them J1 DB25_Socket_MountingHoles, J2 SST39SF040, J3 Adafruit 232H, J4 Altera JTAG, J5 Select 5v, U1 EPM7064STC44-10, X1 ASDMB-xxxMHz

Commit message: Add files via upload
Parts:
- X1: footprint Oscillator:Oscillator_SMD_Abracon_ASDMB-4Pin_2.5x2.0mm -> Oscillator:Oscillator_SMD_Abracon_ASV-4Pin_7.0x5.1mm
- moved X1 1.57 mm to (181.8, 100.0)
- moved C5 0.56 mm to (179.5, 94.5)
Routing:
- net /ROM_WR: track 19.1 -> 22.8 mm
- net /clk_40: track 10.9 -> 7.48 mm
- net GND: track 15.9 -> 18.8 mm
- net +5V: track 197.2 -> 199.6 mm
- net /ROM_OE: track 23.7 -> 25.6 mm
Other:
- board size 53.5 x 34.9 mm -> 53.5 x 37.1 mm
- board text added: "CTX314CT-ND 40Mhz"
- board text added: "EPM7064STC44-10"
- board text added: "SST39SF010A"

Commit message: Add files via upload
Parts:
- moved J5 1.04 mm to (181.0, 90.8)
- moved J4 0.67 mm to (169.8, 89.1)
Routing:
- net /TDI: track 38.8 -> 40.1 mm
- net /TDO: track 36.7 -> 37.9 mm
- net /TMS: track 55.2 -> 55.9 mm
Other:
- board size 53.5 x 37.1 mm -> 53.5 x 38.1 mm

Commit message: Add files via upload
Parts:
- added REF**: MountingHole_2.1mm, MountingHole:MountingHole_2.1mm, F.Cu at (167.7, 104.6)
- moved J5 2.45 mm to (182.0, 88.5)
- moved J4 1.38 mm to (169.8, 87.7)
Routing:
- net +5V: track 199.5 -> 204.3 mm
- net /D5: track 72.7 -> 70.7 mm
- net /D4: track 62.8 -> 61.0 mm
- net /TMS: track 55.9 -> 57.5 mm
- net /D3: track 59.2 -> 57.6 mm
- net /TDI: track 40.1 -> 41.1 mm
- net /TCK: track 40.1 -> 41.0 mm
Other:
- board size 53.5 x 38.1 mm -> 53.5 x 40.6 mm
- board text added: "21FX"
- board text added: "JTAG"
- board text added: "Select 5V"

Commit message: Add files via upload
Routing:
- net /PA1: track 48.9 -> 49.7 mm
- net /PA0: track 47.7 -> 48.3 mm
